File: Hardware/Production/ThingPlus_Micromod-Panel.brd (EAGLE design)
At the start: 203.5 x 130.6 mm, 1446 parts, among them J1 MICROMOD-2222-C, J11 QWIIC_RIGHT_ANGLE, J12 MICRO-SD-SDIOPUSH-PUSH, J13 MICROMOD-2222-C, J16 JTAG, J19 QWIIC_RIGHT_ANGLE, J20 MICRO-SD-SDIOPUSH-PUSH, J21 MICROMOD-2222-C, J24 JTAG, J27 QWIIC_RIGHT_ANGLE, J28 MICRO-SD-SDIOPUSH-PUSH, J29 MICROMOD-2222-C, J32 JTAG, J35 QWIIC_RIGHT_ANGLE, J36 MICRO-SD-SDIOPUSH-PUSH, J37 MICROMOD-2222-C, J4 MICRO-SD-SDIOPUSH-PUSH, J40 JTAG, J43 QWIIC_RIGHT_ANGLE, J44 MICRO-SD-SDIOPUSH-PUSH, J45 MICROMOD-2222-C, J48 JTAG, J51 QWIIC_RIGHT_ANGLE, J52 MICRO-SD-SDIOPUSH-PUSH, J53 MICROMOD-2222-C, J56 JTAG, J59 QWIIC_RIGHT_ANGLE, J60 MICRO-SD-SDIOPUSH-PUSH, J61 MICROMOD-2222-C, J64 JTAG, J67 QWIIC_RIGHT_ANGLE, J68 MICRO-SD-SDIOPUSH-PUSH, J69 MICROMOD-2222-C, J7 QWIIC_RIGHT_ANGLE, J72 JTAG, J75 QWIIC_RIGHT_ANGLE, J76 MICRO-SD-SDIOPUSH-PUSH, J77 MICROMOD-2222-C, J8 JTAG, J80 JTAG, U1 MAX17048, U10 3.3V, U11 AP7361C-33, U12 MCP73831, U13 MAX17048, U14 3.3V, U15 AP7361C-33, U16 MCP73831, U17 MAX17048, U18 3.3V, U19 AP7361C-33, U2 3.3V, U20 MCP73831, U21 MAX17048, U22 3.3V, U23 AP7361C-33, U24 MCP73831, U25 MAX17048, U26 3.3V, U27 MCP73831, U28 AP7361C-33, U29 MCP73831, U3 AP7361C-33, U30 MAX17048, U31 3.3V, U32 AP7361C-33, U33 MCP73831, U34 MAX17048, U35 MAX17048, U36 3.3V, U37 AP7361C-33, U38 MCP73831, U4 MCP73831, U44 3.3V, U5 MAX17048, U6 3.3V, U64 AP7361C-33, U7 AP7361C-33, U8 MCP73831, U9 MAX17048

Commit message: Fixed panel
Parts:
- moved E$3 7.62 mm to (184.1, 118.4)
- moved E$4 7.62 mm to (184.1, 118.4)
- moved D21 2.54 mm to (137.7, 38.6)
- moved D33 2.54 mm to (137.7, 62.0)
- moved D45 2.54 mm to (137.7, 85.3)
- moved D57 2.54 mm to (137.7, 108.7)
- moved D9 2.54 mm to (137.7, 15.2)
- moved H10 2.54 mm to (180.5, 7.49)
- moved H20 2.54 mm to (180.5, 30.9)
- moved H30 2.54 mm to (180.5, 54.2)
- moved H40 2.54 mm to (180.5, 77.6)
- moved H50 2.54 mm to (180.5, 101.0)
- moved J16 2.54 mm to (173.2, 2.54)
- moved J32 2.54 mm to (173.2, 25.9)
- moved J48 2.54 mm to (173.2, 49.3)
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Other:
- board size 203.5 x 130.6 mm -> 211.1 x 130 mm
- board text added: "Route Out"
